File: digicamera/digicamera.kicad_sch (KiCad schematic)
At the start: 71 parts, among them J10 d5, J11 d1, J12 vsync, J13 sda, J14 d2, J15 d6, J16 dclk, J17 d4, J18 d0, J19 scl, J2 mic, J20 href, J21 d3, J22 d7, J23 pclk, J24 xclk, J25 d8, J26 d9, J27 Micro_SD_Card, J3 24 pin 1mm pitch fpc for ov26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, J4 tft touchscreen display, J5 soutp, J6 soutn, J7 Conn_01x05_Pin, J8 Conn_01x05_Pin, J9 Conn_01x05_Pin, SW1 Power Sw, U1 MT3608_DC-DC_STEP_UP_CONVERTE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, U2 MAX98357A, U3 ESP32-S3-DEVKITC-1-N16R8V, U4 MAX4466_Mic_and_Pre-Amp_Audio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, U5 ip2312_module, U6 MIC5365-1.2YC5, U7 MIC5504-2.8YM5

Commit message: finished pcb v1
Parts:
- removed J10: d5, symbol Connector:Conn_01x02_Pin
- removed J11: d1, symbol Connector:Conn_01x02_Pin
- removed J12: vsync, symbol Connector:Conn_01x02_Pin
- removed J13: sda, symbol Connector:Conn_01x02_Pin
- removed J14: d2, symbol Connector:Conn_01x02_Pin
- removed J15: d6, symbol Connector:Conn_01x02_Pin
- removed J16: dclk, symbol Connector:Conn_01x02_Pin
- removed J17: d4, symbol Connector:Conn_01x02_Pin
- removed J18: d0, symbol Connector:Conn_01x02_Pin
- removed J19: scl, symbol Connector:Conn_01x02_Pin
- removed J2: mic, symbol Connector:Conn_01x02_Pin
- removed J20: href, symbol Connector:Conn_01x02_Pin
- removed J21: d3, symbol Connector:Conn_01x02_Pin
- removed J22: d7, symbol Connector:Conn_01x02_Pin
- removed J23: pclk, symbol Connector:Conn_01x02_Pin
- removed J24: xclk, symbol Connector:Conn_01x02_Pin
- removed J25: d8, symbol Connector:Conn_01x02_Pin
- removed J26: d9, symbol Connector:Conn_01x02_Pin
- removed J5: soutp, symbol Connector:Conn_01x02_Pin
- removed J6: soutn, symbol Connector:Conn_01x02_Pin
- added C25: 15p, Capacitor_SMD:C_0805_2012Metric, symbol Device:C
- added C26: 0.1u, Capacitor_SMD:C_0805_2012Metric, symbol Device:C
- added J1, J10, J11, J12, J13, J14, J15, J16, J17, J18, J19, J2, J20, J21, J22, J23, J28, J29, J30, J31, J32, J33, J34, J35, J37, J5, J6: Conn_01x01_Pin, Connector_PinHeader_2.54mm:PinHeader_1x01_P2.54mm_Vertical, symbol Connector:Conn_01x01_Pin
- added R10, R8, R9: 4.7k, Resistor_SMD:R_0805_2012Metric, symbol Device:R
- added R7: 1k, Resistor_SMD:R_0805_2012Metric, symbol Device:R
- added RV1, RV2, RV3, RV4, RV5: 10k, Potentiometer_THT:Potentiometer_Bourns_3386P_Vertical, symbol Device:R_Potentiometer
- BT1, LS1: footprint (none) -> Connector_JST:JST_PH_S2B-PH-K_1x02_P2.00mm_Horizontal
- C1, C10, C11, C12, C13, C14, C15, C16, C17, C18, C19, C2, C20, C21, C22, C23, C24, C3, C4, C5, C6, C7, C8, C9: footprint (none) -> Capacitor_SMD:C_0805_2012Metric
- FB1, FB2: footprint (none) -> ferrite murata BLM21PG600SN1D:BEADC2012X105N
- J27: footprint (none) -> Connector_Card:microSD_HC_Hirose_DM3AT-SF-PEJM5
- J3: footprint (none) -> Connector_FFC-FPC:Molex_200528-0240_1x24-1MP_P1.00mm_Horizontal
- J4: footprint (none) -> Connector_PinHeader_2.54mm:PinHeader_1x14_P2.54mm_Vertical
- J7, J8, J9: footprint (none) -> Connector_PinHeader_2.54mm:PinHeader_1x05_P2.54mm_Vertical
- R1: footprint (none) -> Resistor_SMD:R_0805_2012Metric
- R2, R3, R4, R5, R6: value 10k -> 47k; footprint (none) -> Resistor_SMD:R_0805_2012Metric
- SW1: footprint (none) -> RLS-102-F1-Miniature Rocker Toggle:RLS-102-F1-Toggle
- U1: footprint MT3608_DC-DC_STEP_UP_CONVERTER_2A_BOOSTER_MODULE:MODULE_MT3608_DC-DC_STEP_UP_CONVERTER_2A_BOOSTER_MODULE -> mt3608_module:MODULE_MT3608_DC-DC_STEP_UP_CONVERTER_2A_BOOSTER_MODULE
- U2: footprint (none) -> max98357a_ic:QFN50P300X300X80-17N
- U3: footprint (none) -> esp32s3_devkit:XCVR_ESP32-S3-DEVKITC-1-N16R8V
- U4: footprint (none) -> max4466_withmic_evalboard:MODULE_MAX4466_Microphone_Pre-Amp_Audio_Evaluation_Board
- U5: footprint (none) -> ip2312_module:Untitled
Connections:
- net dgnd is gone; now on net GND: J3.10 (Pin_10)
- net gain is gone; now on net GND: U2.2 (GAIN_SLOT)
- net led1_data is gone; now on net led_data: D5.4 (DIN)
- net led2_data is gone; now on an unnamed net: D6.4 (DIN)
- net led3_data is gone; now on an unnamed net: D7.4 (DIN)
- net sdmiso is gone; now on net lcdmiso: J27.7 (DAT0), R4.2
- net sdmosi is gone; now on net lcdmosi: J27.3 (CMD), R2.2
- net sdsck is gone; now on net lcdsck: J27.5 (CLK)
- net t_clk is gone; now on net lcdsck: J4.10 (Pin_10)
- net t_din is gone; now on net lcdmosi: J4.12 (Pin_12)
- net t_do is gone; now on net lcdmiso: J4.13 (Pin_13)
- net +3V3: now also R10.2, R8.2, R9.2
- net GND: now also J3.MP, C25.2, C26.2, R7.2, RV1.3, RV2.3, RV3.3, RV4.3, RV5.3
- net bclk: now also U3.J1_20 (GPIO14)
- net d2: now also U3.J1_7 (GPIO7), J17.1 (Pin_1)
- net d3: now also U3.J1_5 (GPIO5), J19.1 (Pin_1)
- net d4: now also U3.J1_4 (GPIO4), J23.1 (Pin_1)
- net d5: now also U3.J1_6 (GPIO6), J10.1 (Pin_1)
- net d6: now also U3.J1_8 (GPIO15), J18.1 (Pin_1)
- net d7: now also U3.J1_10 (GPIO17), J14.1 (Pin_1)
- net d8: now also U3.J1_11 (GPIO18), J12.1 (Pin_1)
- net d9: now also U3.J1_15 (GPIO9), J11.1 (Pin_1)
- net din: now also U3.J3_17 (GPIO47)
- net href: now also U3.J1_16 (GPIO10), J20.1 (Pin_1)
- net lcdcs: now also U3.J3_2 (U0TXD/GPIO43)
- net lcddc/rs: now also U3.J3_5 (GPIO2)
- net lcdmiso: now also U3.J3_7 (MTDI/GPIO41)
- net lcdmosi: now also U3.J3_8 (MTDO/GPIO40)
- net lcdrst: now also U3.J3_10 (GPIO38)
- net lcdsck: now also U3.J3_9 (MTCK/GPIO39)
- net lrclk: now also U3.J3_16 (GPIO48)
- net mic: now also U3.J3_4 (GPIO1), J22.1 (Pin_1)
- net pclk: now also U3.J1_9 (GPIO16), C25.1, J5.1 (Pin_1)
- net pwdn: now also R7.1
- net rstb: now also C26.1, R8.1
- net scl: now also U3.J1_18 (GPIO12), J21.1 (Pin_1), R10.1
- net sda: now also U3.J1_19 (GPIO13), J16.1 (Pin_1), R9.1
- net sdcs: now also U3.J3_6 (MTMS/GPIO42)
- net soutn: now also J13.1 (Pin_1)
- net soutp: now also J6.1 (Pin_1)
- net t_cs: now also U3.J3_3 (U0RXD/GPIO44)
- net t_irq: now also U3.J3_18 (GPIO21)
- net vsync: now also U3.J1_17 (GPIO11), J15.1 (Pin_1)
- net xclk: now also U3.J1_12 (GPIO8), J2.1 (Pin_1)
- net led_data: now reaches U3.J3_14 (GPIO0)
- new net: J31.1 (Pin_1), RV3.1
- new net: J33.1 (Pin_1), RV3.2
- new net: J35.1 (Pin_1), RV5.1
- new net: J30.1 (Pin_1), RV2.2
- new net: J29.1 (Pin_1), RV2.1
- new net: J34.1 (Pin_1), RV4.2
- new net: J32.1 (Pin_1), RV4.1
- new net: J37.1 (Pin_1), RV5.2
- new net: J28.1 (Pin_1), RV1.1
- new net: J1.1 (Pin_1), RV1.2
- no-connect marks 5 -> 16
Other:
- note added: "10k trimpot"
- note added: "toggle"
- note removed: "pinouts"
- moved on the sheet: BT1, C1, C10, C11, C12, C13, C14, C15, C16, C17, C18, C19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
